File: controller_from_scratch.kicad_sch (KiCad schematic)
At the start: 0 parts

Commit message: this is some stuff
Parts:
- added J1: USB_C_Receptacle_USB2.0_14P, symbol Connector:USB_C_Receptacle_USB2.0_14P
- added R1: 5.1K, symbol Device:R
- added R2: 5.1k, symbol Device:R
- added SW1, SW2, SW3, SW4: SW_Push, symbol Switch:SW_Push
- added U1: ESP32-C3-WROOM-02, RF_Module:ESP32-C3-WROOM-02, symbol RF_Module:ESP32-C3-WROOM-02
Connections:
- new net: J1.B5 (CC2), R1.1
- new net: J1.A5 (CC1), R2.1
- new net +3V3: U1.1 (3V3), U1.2 (EN)
- new net +5V: J1.A4 (VBUS), J1.A9 (VBUS), J1.B4 (VBUS), J1.B9 (VBUS)
- new net GND: J1.A1 (GND), J1.A12 (GND), J1.B1 (GND), J1.B12 (GND), J1.SH (SHIELD), R1.2, R2.2, U1.19 (GND), U1.9 (GND)
- new net IO18: J1.A7 (D-), J1.B7 (D-), U1.13 (IO18)
- new net IO19: J1.A6 (D+), J1.B6 (D+), U1.14 (IO19)

Commit message: commit of work for right now
Parts:
- removed SW1, SW2, SW3, SW4: SW_Push, symbol Switch:SW_Push
- added C1, C2: 10uF, symbol Device:C
- added C3, C4, C6: 100nF, symbol Device:C
- added C5: C, symbol Device:C
- added D1, D2, D3, D4, D5, D6, D7, D8, D9: D, symbol Device:D
- added JOY1, JOY2: (no value), symbol KY-023:KY-023
- added R3, R4, R5, R6: 10K, symbol Device:R
- added R7: R, symbol Device:R
- added R8, R9: 4.7K, symbol Device:R
- added SW1, SW10, SW11, SW2, SW3, SW4, SW7, SW8, SW9: SW_Push_45deg, symbol Switch:SW_Push_45deg
- added SW12, SW13, SW14, SW15, SW5, SW6: SW_Push, symbol Switch:SW_Push
- added U2: LD1117S33TR_SOT223, Package_TO_SOT_SMD:SOT-223-3_TabPin2, symbol Regulator_Linear:LD1117S33TR_SOT223
- added U3: MCP23017x-x-SO, Package_SO:SOIC-28W_7.5x17.9mm_P1.27mm, symbol Interface_Expansion:MCP23017x-x-SO
Connections:
- net +3V3: now also C2.2, C3.2, R3.1, R4.1, R5.1, R6.1, R8.1, R9.2, U2.2 (VO); no longer U1.2 (EN)
- net +5V: now also C1.1, C5.2, JOY1.1 (+5V), JOY2.1 (+5V), U2.3 (VI)
- net GND: now also C1.2, C2.1, C3.1, C4.1, C5.1, C6.1, JOY1.0 (GND), JOY2.0 (GND), SW12.1, SW13.1, SW14.1, SW15.1, SW5.1, SW6.2, U2.1 (GND), U3.10 (V_{SS}), U3.15 (A0), U3.16 (A1), U3.17 (A2)
- net Row3: now reaches U1.10 (IO10)
- net Row3: now also SW10.1, SW11.1, SW9.1
- net JOY_1_B: now reaches U1.11 (IO20/RXD)
- net at U1.16 (IO2): now also R4.2
- net JOY_2_Y: now reaches U1.17 (IO1)
- net JOY_2_Y: now also JOY2.3 (VRY)
- net JOY_2_X: now reaches U1.18 (IO0)
- net JOY_2_X: now also JOY2.2 (VRX)
- net JOY_1_X: now reaches U1.3 (IO4)
- net JOY_1_X: now also JOY1.2 (VRX)
- net JOY_1_Y: now reaches U1.4 (IO5)
- net JOY_1_Y: now also JOY1.3 (VRY)
- net CLOCK: now reaches U1.5 (IO6)
- net CLOCK: now also R9.1, U3.12 (SCK)
- net DATA: now reaches U1.6 (IO7)
- net DATA: now also R8.2, U3.13 (SDA)
- net at U1.7 (IO8): now also R3.2
- net at U1.8 (IO9): now also R5.2, SW5.2
- net IO18 renamed D-
- net IO19 renamed D+
- new net: C4.2, R7.1, SW6.1
- new net: D3.2 (A), SW11.2
- new net: D4.2 (A), SW8.2
- new net: C6.2, U3.9 (V_{DD})
- new net: D9.2 (A), SW3.2
- new net: D6.2 (A), SW4.2
- new net: D7.2 (A), SW1.2
- new net: D8.2 (A), SW2.2
- new net: D5.2 (A), SW7.2
- new net: D2.2 (A), SW10.2
- new net: R6.2, U3.18 (~{RESET})
- new net: D1.2 (A), SW9.2
- new net EN: R7.2, U1.2 (EN)
- new net JOY_A: JOY2.4 (SW), U3.21 (GPA0)
- new net JOY_B: JOY1.4 (SW)
- new net Row1: SW1.1, SW2.1, SW3.1, U3.26 (GPA5)
- new net Row2: SW4.1, SW7.1, SW8.1, U3.25 (GPA4)
- new net Row4: D1.1 (K), D6.1 (K), D7.1 (K), U3.23 (GPA2)
- new net Row5: D2.1 (K), D5.1 (K), D8.1 (K), U3.22 (GPA1)
- new net Row6: D3.1 (K), D4.1 (K), D9.1 (K), U3.24 (GPA3)
- new net TRIGGER_LEFT_A: SW13.2, U3.27 (GPA6)
- new net TRIGGER_LEFT_B: SW12.2, U3.28 (GPA7)
- new net TRIGGER_RIGHT_A: SW14.2, U3.1 (GPB0)
- new net TRIGGER_RIGHT_B: SW15.2, U3.2 (GPB1)
- no-connect marks 0 -> 8
Other:
- note added: "Regular Buttons"
- note added: "This must be the bottom joystick"
- moved on the sheet: U1

Commit message: finished pcb design
Parts:
- removed C5: C, symbol Device:C
- removed JOY2: (no value), symbol KY-023:KY-023
- added JOY3: (no value), Connector_PinHeader_2.54mm:PinHeader_1x05_P2.54mm_Vertical, symbol KY-023:KY-023
- C1, C2, C3, C4, C6: footprint (none) -> Capacitor_SMD:C_1206_3216Metric
- D1, D2, D3, D4, D5, D6, D7, D8, D9: footprint (none) -> Diode_SMD:D_1206_3216Metric_Pad1.42x1.75mm_HandSolder
- J1: footprint (none) -> Connector_USB:USB_C_Receptacle_HRO_TYPE-C-31-M-12
- JOY1: footprint (none) -> Connector_PinHeader_2.54mm:PinHeader_1x05_P2.54mm_Vertical
- R1, R2, R3, R4, R5, R6: footprint (none) -> Resistor_SMD:R_1206_3216Metric_Pad1.30x1.75mm_HandSolder
- R7: value R -> 10k; footprint (none) -> Resistor_SMD:R_1206_3216Metric_Pad1.30x1.75mm_HandSolder
- R8, R9: value 4.7K -> 10K; footprint (none) -> Resistor_SMD:R_1206_3216Metric_Pad1.30x1.75mm_HandSolder
- SW1, SW10, SW11, SW12, SW13, SW14, SW15, SW2, SW3, SW4, SW5, SW6, SW7, SW8, SW9: footprint (none) -> Connector_PinHeader_2.54mm:PinHeader_2x01_P2.54mm_Vertical
Connections:
- net JOY_1_B is gone; now on net JOY_B: U1.11 (IO20/RXD)
- net +3V3: now also C6.2, R7.1, U3.9 (V_{DD})
- net +5V: no longer JOY1.1 (+5V)
- net EN: now also C4.2, SW6.1
- net GND: now also JOY1.1 (GND), JOY3.1 (GND); no longer JOY1.0 (GND)
- net JOY_1_X: now also JOY3.3 (VRX); no longer JOY1.2 (VRX)
- net JOY_1_Y: now also JOY3.4 (VRY); no longer JOY1.3 (VRY)
- net JOY_2_X: now also JOY1.3 (VRX)
- net JOY_2_Y: now also JOY1.4 (VRY)
- net JOY_A: now also JOY1.5 (SW)
- net JOY_B: now also JOY3.5 (SW); no longer JOY1.4 (SW)
- new net +3.3V: JOY1.2 (+5V), JOY3.2 (+5V)
- no-connect marks 8 -> 10
Other:
- note removed: "This must be the bottom joystick"
- moved on the sheet: C4, SW6
